File: stir_plate1.brd (EAGLE design)
At the start: 100 x 80 mm, 10 parts, among them U1 V_REG_317SINK

Commit message: changes
Parts:
- moved JP2 92.7 mm to (96.5, 10.2)
- moved U1 78.8 mm to (94.0, 24.1), turned to 270 degrees
- moved R1 62.2 mm to (80.0, 1.27)
- moved R3 61.0 mm to (20.3, 1.27)
- moved JP3 14.0 mm to (81.3, 33.0), turned to 180 degrees
- moved ULN1 13.5 mm to (49.5, 7.62), turned to 0 degrees
- moved U$1 9.67 mm to (35.6, 26.7), turned to 270 degrees
- moved JP4 9.16 mm to (81.3, 26.7), turned to 90 degrees
Routing:
- net VCC: track 187.9 -> 67.2 mm
- net N$2: track 61.1 -> 0.00 mm
- net N$15: track 0.00 -> 57.1 mm
- net N$6: track 0.00 -> 55.3 mm
- net N$14: track 0.00 -> 48.6 mm
- net N$3: track 106.5 -> 65.6 mm
- net N$12: track 20.9 -> 56.3 mm
- net N$1: track 0.00 -> 25.4 mm
- net N$8: track 258.1 -> 282.3 mm
- net N$13: track 46.4 -> 62.7 mm
- net N$10: track 56.3 -> 41.0 mm
- net N$9: track 53.5 -> 41.0 mm
- net N$11: track 44.9 -> 57.0 mm
- net N$7: track 51.6 -> 41.0 mm
- net GND: track 271.5 -> 280.9 mm
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